File: Hardware/LEDTischLampe.kicad_pcb (KiCad board)
At the start: 2 copper layers, 160 x 160 mm, 119 parts, among them J1 Conn_01x02_Socket, J2 USB_C_Receptacle_USB2.0_14P, J3 Conn_02x03_Counter_Clockwise, Q1 P-CHANNEL-MOSFET, SW1 Reset, SW2 User, U1 ESP32-C3-WROOM-02, U3 SY7200AABC, U4 SY7200AABC, U5 SY7200AABC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

Commit message: final touches for v1.0
Parts:
- removed D34: 15V, Diode_SMD:D_0402_1005Metric
- removed Q1: P-CHANNEL-MOSFET, Package_SON:VSON-8_3.3x3.3mm_P0.65mm_NexFET
- removed R17: 100k, Resistor_SMD:R_0402_1005Metric
- added D25: SS34, Diode_SMD:D_SMA, F.Cu at (134.6, 122.4)
- C10, C11, C12, C18, C2, C6, C9: footprint Capacitor_SMD:C_1210_3225Metric -> Capacitor_SMD:C_0805_2012Metric
- moved C18 1.09 mm to (149.5, 77.1)
- moved C2 0.79 mm to (118.4, 113.4)
- moved ? 0.63 mm to (92.8, 92.2)
- moved C10 0.59 mm to (146.6, 41.3)
- moved C12 0.50 mm to (144.4, 141.1)
- moved C9 0.50 mm to (170.6, 133.0)
- moved C11 0.42 mm to (158.9, 139.7)
- moved C25 0.38 mm to (147.8, 77.6)
Connections:
- J1 pad 1: Net-(J1-Pin_1) -> VCC
Routing:
- net VCC: track 23.6 -> 29.2 mm
- net Net-(D34-A): track 2.57 -> 0.00 mm
- net +3V3: track 108.6 -> 106.1 mm
- net GND: track 69.3 -> 69.8 mm, vias 42 -> 41
- removed copper zone on F.Cu, net Net-(J1-Pin_1)

Commit message: some more tweaks (rotated input terminal block, added voltage measurement)
Parts:
- added C13: 100n, Capacitor_SMD:C_0402_1005Metric, F.Cu at (151.6, 70.2)
- added G***: LOGO, LOGO, F.Cu at (118.1, 82.8)
- added R17: 47k, Resistor_SMD:R_0402_1005Metric, F.Cu at (151.1, 68.7)
- added R18: 4k7, Resistor_SMD:R_0402_1005Metric, F.Cu at (150.6, 70.2)
- moved J1 5.04 mm to (137.1, 114.3), turned to 180 degrees
Connections:
- J1 pad 1: VCC -> GND
- J1 pad 2: GND -> VCC
- U1 pad 3: unconnected-(U1-IO4-Pad3) -> V_{sense}
Routing:
- net V_{sense}: track 0.00 -> 15.3 mm
- net GND: track 69.8 -> 71.5 mm, vias 41 -> 42
Other:
- board text added: "Boot"
- board text added: "Reset"

Commit message: update RGB mapping in KiCad
Connections:
- net /LedsOben/LedTreiber1/LEDN renamed /LedsOben/LedTreiberB/LEDN
- net /LedsOben/LedTreiber1/LEDP renamed /LedsOben/LedTreiberB/LEDP
- net /LedsOben/LedTreiber2/LEDN renamed /LedsOben/LedTreiberR/LEDN
- net /LedsOben/LedTreiber2/LEDP renamed /LedsOben/LedTreiberR/LEDP
- net /LedsOben/LedTreiber3/LEDN renamed /LedsOben/LedTreiberG/LEDN
- net /LedsOben/LedTreiber3/LEDP renamed /LedsOben/LedTreiberG/LEDP
- C4 pad 2: Net-(U7-SW) -> Net-(C4-Pad2)
- L1 pad 1: Net-(U7-SW) -> Net-(C4-Pad2)
- U1 pad 15: RDim -> BDim
- U1 pad 16: GDim -> RDim
- U1 pad 17: BDim -> GDim
- U4 pad 4: RDim -> BDim
- U5 pad 4: GDim -> RDim
- U6 pad 4: BDim -> GDim
- U7 pad 6: Net-(U7-SW) -> unconnected-(U7-SW-Pad6)
Routing:
- net BDim: track 105.3 -> 128.3 mm
- net GDim: track 122.8 -> 105.3 mm
- net RDim: track 128.3 -> 122.8 mm
- added copper zone on F.Cu, net Net-(C4-Pad2)
- removed copper zone on F.Cu, net Net-(U7-SW)
Other:
- board text added: "G R B"
- board text added: "W"
